Commit message: Final Project

File: my_robot_description/urdf/common_properties.urdf.xacro (robot description, xacro)
@@ -10,3 +10,30 @@
         <color rgba="0.5 0.5 0.5 1"></color>
     </material>
+    <xacro:macro name="box_inertia" params="mass length width height xyz rpy">
+        <inertial>
+            <origin xyz="${xyz}" rpy="${rpy}"></origin>
+            <mass value="${mass}"></mass>
+            <inertia ixx="${(mass/12)*(height*height + length*length)}" ixy="0" ixz="0"
+                     iyy="${(mass/12)*(width*width + length*length)}" iyz="0"
+                     izz="${(mass/12)*(width*width + height*height)}"></inertia>
+        </inertial>
+    </xacro:macro>
+    <xacro:macro name="cylinder_inertia" params="mass length radius xyz rpy">
+        <inertial>
+            <origin xyz="${xyz}" rpy="${rpy}"></origin>
+            <mass value="${mass}"></mass>
+            <inertia ixx="${(mass/12)*(3*radius*radius + length*length)}" ixy="0" ixz="0"
+                     iyy="${(mass/12)*(3*radius*radius + length*length)}" iyz="0"
+                     izz="${(mass/2)*(radius*radius)}"></inertia>
+        </inertial>
+    </xacro:macro>
+    <xacro:macro name="sphere_inertia" params="mass radius xyz rpy">
+        <inertial>
+            <origin xyz="${xyz}" rpy="${rpy}"></origin>
+            <mass value="${mass}"></mass>
+            <inertia ixx="${(2*mass/5)*radius*radius}" ixy="0" ixz="0"
+                     iyy="${(2*mass/5)*radius*radius}" iyz="0"
+                     izz="${(2*mass/5)*radius*radius}"></inertia>
+        </inertial>
+    </xacro:macro>
 </robot>

File: my_robot_description/urdf/mobile_base.urdf.xacro (robot description, xacro)
@@ -6,6 +6,5 @@
     <xacro:property name="wheel_radius" value="0.1"></xacro:property>
     <xacro:property name="wheel_length" value="0.05"></xacro:property>
-    <link name="base_footprint">
-    </link>
+    <link name="base_footprint"></link>
     <link name="base_link">
         <visual>
@@ -16,14 +15,32 @@
             <material name="green"></material>
         </visual>
+        <collision>
+            <geometry>
+                <box size="${base_length} ${base_width} ${base_height}"></box>
+            </geometry>
+            <origin xyz="0 0 ${base_height/2.0}" rpy="0 0 0"></origin>
+        </collision>
+        <xacro:box_inertia mass="5.0" length="${2*base_length}" width="${2*base_width}"
+                           height="${2*base_height}" xyz="0 0 ${base_height/2.0}" rpy="0 0 0">
+        </xacro:box_inertia>
     </link>
     <xacro:macro name="wheel_link" params="prefix">
         <link name="${prefix}_wheel_link">
             <visual>
-            <geometry>
-                <cylinder radius="${wheel_radius}" length="${wheel_length}"></cylinder>
-            </geometry>
-            <origin xyz="0 0 0" rpy="${pi/2.0} 0 0"></origin>
-            <material name="grey"></material>
-        </visual>
+                <geometry>
+                    <cylinder radius="${wheel_radius}" length="${wheel_length}"></cylinder>
+                </geometry>
+                <origin xyz="0 0 0" rpy="${pi/2.0} 0 0"></origin>
+                <material name="grey"></material>
+            </visual>
+            <collision>
+                <geometry>
+                    <cylinder radius="${wheel_radius}" length="${wheel_length}"></cylinder>
+                </geometry>
+                <origin xyz="0 0 0" rpy="${pi/2.0} 0 0"></origin>
+            </collision>
+            <xacro:cylinder_inertia mass="1.0" radius="${2*wheel_radius}" length="${2*wheel_length}"
+                                    xyz="0 0 0" rpy="${pi/2.0} 0 0">
+            </xacro:cylinder_inertia>
         </link>
     </xacro:macro>
@@ -38,4 +55,12 @@
             <material name="grey"></material>
         </visual>
+        <collision>
+            <geometry>
+                <sphere radius="${wheel_radius/2.0}"></sphere>
+            </geometry>
+            <origin xyz="0 0 0" rpy="0 0 0"></origin>
+        </collision>
+        <xacro:sphere_inertia mass="0.5" radius="${wheel_radius}" xyz="0 0 0" rpy="0 0 0">
+        </xacro:sphere_inertia>
     </link>
     <joint name="base_right_wheel_joint" type="continuous">

File: my_robot_description/urdf/my_robot.urdf.xacro (robot description, xacro)
@@ -3,3 +3,5 @@
     <xacro:include filename="common_properties.urdf.xacro"></xacro:include>
     <xacro:include filename="mobile_base.urdf.xacro"></xacro:include>
+    <xacro:include filename="mobile_base_gazebo.urdf.xacro"></xacro:include>
+    <xacro:include filename="camera.urdf.xacro"></xacro:include>
 </robot>

Commit message: Course completed

File: my_robot_description/urdf/common_properties.urdf.xacro (robot description, xacro)
@@ -9,4 +9,10 @@
     <material name="grey">
         <color rgba="0.5 0.5 0.5 1"></color>
+    </material>
+    <material name="yellow">
+        <color rgba="1 1 0 1"></color>
+    </material>
+    <material name="orange">
+        <color rgba="1 0.5 0 1"></color>
     </material>
     <xacro:macro name="box_inertia" params="mass length width height xyz rpy">

File: my_robot_description/urdf/mobile_base.urdf.xacro (robot description, xacro)
@@ -64,4 +64,9 @@
         </xacro:sphere_inertia>
     </link>
+    <joint name="base_joint" type="fixed">
+        <parent link="base_footprint"></parent>
+        <child link="base_link"></child>
+        <origin xyz="0 0 ${base_height/2}" rpy="0 0 0"></origin>
+    </joint>
     <joint name="base_right_wheel_joint" type="continuous">
         <parent link="base_link"></parent>
@@ -81,8 +86,3 @@
         <origin xyz="${base_length/3.0} 0 -${wheel_radius/2.0}" rpy="0 0 0"></origin>
     </joint>
-    <joint name="base_joint" type="fixed">
-        <parent link="base_footprint"></parent>
-        <child link="base_link"></child>
-        <origin xyz="0 0 ${base_height/2}" rpy="0 0 0"></origin>
-    </joint>
 </robot>

File: my_robot_description/urdf/my_robot.urdf.xacro (robot description, xacro)
@@ -5,3 +5,10 @@
     <xacro:include filename="mobile_base_gazebo.urdf.xacro"></xacro:include>
     <xacro:include filename="camera.urdf.xacro"></xacro:include>
+    <xacro:include filename="arm.xacro"></xacro:include>
+    <xacro:include filename="arm_gazebo.urdf.xacro"></xacro:include>
+    <joint name="mobile_base_arm_joint" type="fixed">
+        <parent link="base_link"></parent>
+        <child link="arm_base_link"></child>
+        <origin xyz="${base_length/4} 0 ${base_height}" rpy="0 0 0"></origin>
+    </joint>
 </robot>
